Commit message: Updated wheel visuals
Signed-off-by: Mihir Kulkarni <mihirk284@gmail.com>

File: smb_description/urdf/smb.urdf.xacro (robot description, xacro)
@@ -38,5 +38,5 @@
 	</link>
 	<gazebo reference="base_link">
-		<material>Gazebo/Blue</material>
+		<material>Gazebo/Orange</material>
 	</gazebo>
 	<!-- Interial link stores the robot's inertial information -->

File: smb_description/urdf/wheel.urdf.xacro (robot description, xacro)
@@ -3,8 +3,8 @@
     <xacro:property name="PI" value="3.1415926535897931"/>
     <xacro:property name="robot_name" value="smb"/>
-    <xacro:property name="wheelWidth" value="0.17"/>
+    <xacro:property name="wheelWidth" value="0.185"/>
     <xacro:property name="wheelRadius" value="0.19"/>
     <xacro:property name="frontWheelX" value="0.2159"/>
-    <xacro:property name="backWheelX" value="-0.2159"/>
+    <xacro:property name="backWheelX" value="-0.21"/>
     <xacro:property name="wheelClearance" value="0.03"/>
     <xacro:property name="wheelHeight" value="0.05"/>
@@ -21,5 +21,5 @@
 				<geometry>
 					<!-- <cylinder length="${wheelWidth}" radius="${wheelRadius}"/> -->
-					<cylinder length="0.1" radius="0.1"/>  <!-- wheel visual dimensions are small to make the mesh fit properly -->
+					<cylinder length="0.17" radius="0.20"/>  <!-- wheel visual dimensions are small to make the mesh fit properly -->
 				</geometry>
 				<material name="black"/>
